File: production/ecad/FufuS24/Control.kicad_sch (KiCad schematic)
At the start: 28 parts, among them IC1 NLVPCA9535EDTR2G, J2 Conn_01x02, U1 RP2040, U2 W25Q128JVS

Commit message: Final Foot Fetish
Parts:
- U2: footprint Package_SO:SOIC-8_5.23x5.23mm_P1.27mm -> footprints:W25Q128JVSIM_footprint
- Y1: footprint (none) -> footprints:XTAL_ABLS-12.000MHZ-B4-T
Changed lines of the file:
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@@
       (effects (font (size 1.27 1.27)))
     )
-    (property "Footprint" "" (at 75.565 120.65 0)
+    (property "Footprint" "footprints:XTAL_ABLS-12.000MHZ-B4-T" (at 75.565 120.65 0)
       (effects (font (size 1.27 1.27)) hide)
     )
@@
       (effects (font (size 1.27 1.27)))
     )
-    (property "Footprint" "Package_SO:SOIC-8_5.23x5.23mm_P1.27mm" (at 46.355 95.25 0)
+    (property "Footprint" "footprints:W25Q128JVSIM_footprint" (at 46.355 95.25 0)
       (effects (font (size 1.27 1.27)) hide)
     )

Commit message: efan finals before laying out
Connections:
- net I2C0_SCL: now also R29.2
- net I2C0_SDA: now also R19.2
Other:
- moved on the sheet: R19, R29
Changed lines of the file:
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@@
   (junction (at 168.275 35.56) (diameter 0) (color 0 0 0 0)
   )
+  (junction (at 266.065 118.745) (diameter 0) (color 0 0 0 0)
+  )
   (junction (at 125.095 53.34) (diameter 0) (color 0 0 0 0)
   )
@@
   (junction (at 189.865 115.57) (diameter 0) (color 0 0 0 0)
   )
+  (junction (at 264.16 116.205) (diameter 0) (color 0 0 0 0)
+  )
   (junction (at 168.275 43.18) (diameter 0) (color 0 0 0 0)
   )
   (junction (at 156.845 35.56) (diameter 0) (color 0 0 0 0)
   )
-  (junction (at 266.065 60.96) (diameter 0) (color 0 0 0 0)
+  (junction (at 266.7 78.105) (diameter 0) (color 0 0 0 0)
   )
   (junction (at 133.985 35.56) (diameter 0) (color 0 0 0 0)
@@
     (stroke (width 0) (type default))
   )
-  (wire (pts (xy 260.985 63.5) (xy 260.985 60.96))
+  (wire (pts (xy 261.62 80.645) (xy 261.62 78.105))
     (stroke (width 0) (type default))
   )
@@
     (stroke (width 0) (type default))
   )
-  (wire (pts (xy 262.255 118.745) (xy 267.335 118.745))
+  (wire (pts (xy 262.255 118.745) (xy 266.065 118.745))
     (stroke (width 0) (type default))
   )
@@
     (stroke (width 0) (type default))
   )
+  (wire (pts (xy 266.065 88.265) (xy 266.065 118.745))
+    (stroke (width 0) (type default))
+  )
   (wire (pts (xy 179.705 105.41) (xy 179.705 118.11))
     (stroke (width 0) (type default))
@@
     (stroke (width 0) (type default))
   )
-  (wire (pts (xy 262.255 116.205) (xy 267.335 116.205))
-    (stroke (width 0) (type default))
-  )
   (wire (pts (xy 168.275 43.18) (xy 179.705 43.18))
     (stroke (width 0) (type default))
@@
     (stroke (width 0) (type default))
   )
+  (wire (pts (xy 266.065 118.745) (xy 267.335 118.745))
+    (stroke (width 0) (type default))
+  )
   (wire (pts (xy 262.255 126.365) (xy 267.335 126.365))
     (stroke (width 0) (type default))
@@
     (stroke (width 0) (type default))
   )
-  (wire (pts (xy 260.985 60.96) (xy 266.065 60.96))
+  (wire (pts (xy 261.62 78.105) (xy 266.7 78.105))
     (stroke (width 0) (type default))
   )
@@
     (stroke (width 0) (type default))
   )
-  (wire (pts (xy 266.065 60.96) (xy 271.145 60.96))
+  (wire (pts (xy 266.7 78.105) (xy 271.78 78.105))
     (stroke (width 0) (type default))
   )
@@
     (stroke (width 0) (type default))
   )
+  (wire (pts (xy 264.16 116.205) (xy 267.335 116.205))
+    (stroke (width 0) (type default))
+  )
   (wire (pts (xy 117.475 153.67) (xy 117.475 156.21))
     (stroke (width 0) (type default))
@@
     (stroke (width 0) (type default))
   )
+  (wire (pts (xy 264.16 88.265) (xy 264.16 116.205))
+    (stroke (width 0) (type default))
+  )
   (wire (pts (xy 268.605 106.045) (xy 268.605 99.06))
     (stroke (width 0) (type default))
@@
     (stroke (width 0) (type default))
   )
+  (wire (pts (xy 264.16 88.265) (xy 261.62 88.265))
+    (stroke (width 0) (type default))
+  )
   (wire (pts (xy 53.975 62.865) (xy 53.975 65.405))
     (stroke (width 0) (type default))
@@
     (stroke (width 0) (type default))
   )
-  (wire (pts (xy 271.145 60.96) (xy 271.145 63.5))
+  (wire (pts (xy 271.78 78.105) (xy 271.78 80.645))
     (stroke (width 0) (type default))
   )
@@
     (stroke (width 0) (type default))
   )
+  (wire (pts (xy 262.255 116.205) (xy 264.16 116.205))
+    (stroke (width 0) (type default))
+  )
   (wire (pts (xy 142.875 130.81) (xy 161.925 130.81))
     (stroke (width 0) (type default))
@@
   )
   (wire (pts (xy 125.095 31.115) (xy 125.095 35.56))
+    (stroke (width 0) (type default))
+  )
+  (wire (pts (xy 266.065 88.265) (xy 271.78 88.265))
     (stroke (width 0) (type default))
   )
@@
     )
   )
-  (symbol (lib_id "Device:R") (at 271.145 67.31 0) (unit 1)
-    (in_bom yes) (on_board yes) (dnp no) (fields_autoplaced)
-    (property "Reference" "R29" (at 273.685 66.04 0)
-      (effects (font (size 1.27 1.27)) (justify left))
-    )
-    (property "Value" "4.7k" (at 273.685 68.58 0)
-      (effects (font (size 1.27 1.27)) (justify left))
-    )
-    (property "Footprint" "footprints:RESC2012X60N" (at 269.367 67.31 90)
-      (effects (font (size 1.27 1.27)) hide)
-    )
-    (property "Datasheet" "~" (at 271.145 67.31 0)
+  (symbol (lib_id "Device:R") (at 271.78 84.455 0) (unit 1)
+    (in_bom yes) (on_board yes) (dnp no) (fields_autoplaced)
+    (property "Reference" "R29" (at 274.32 83.185 0)
+      (effects (font (size 1.27 1.27)) (justify left))
+    )
+    (property "Value" "4.7k" (at 274.32 85.725 0)
+      (effects (font (size 1.27 1.27)) (justify left))
+    )
+    (property "Footprint" "footprints:RESC2012X60N" (at 270.002 84.455 90)
+      (effects (font (size 1.27 1.27)) hide)
+    )
+    (property "Datasheet" "~" (at 271.78 84.455 0)
       (effects (font (size 1.27 1.27)) hide)
     )
@@
     )
   )
-  (symbol (lib_id "Device:R") (at 260.985 67.31 0) (unit 1)
-    (in_bom yes) (on_board yes) (dnp no) (fields_autoplaced)
-    (property "Reference" "R19" (at 263.525 66.04 0)
-      (effects (font (size 1.27 1.27)) (justify left))
-    )
-    (property "Value" "4.7k" (at 263.525 68.58 0)
-      (effects (font (size 1.27 1.27)) (justify left))
-    )
-    (property "Footprint" "footprints:RESC2012X60N" (at 259.207 67.31 90)
-      (effects (font (size 1.27 1.27)) hide)
-    )
-    (property "Datasheet" "~" (at 260.985 67.31 0)
+  (symbol (lib_id "Device:R") (at 261.62 84.455 0) (unit 1)
+    (in_bom yes) (on_board yes) (dnp no) (fields_autoplaced)
+    (property "Reference" "R19" (at 264.16 83.185 0)
+      (effects (font (size 1.27 1.27)) (justify left))
+    )
+    (property "Value" "4.7k" (at 264.16 85.725 0)
+      (effects (font (size 1.27 1.27)) (justify left))
+    )
+    (property "Footprint" "footprints:RESC2012X60N" (at 259.842 84.455 90)
+      (effects (font (size 1.27 1.27)) hide)
+    )
+    (property "Datasheet" "~" (at 261.62 84.455 0)
       (effects (font (size 1.27 1.27)) hide)
     )
@@
     )
   )
-  (symbol (lib_id "power:+3.3V") (at 266.065 60.96 0) (unit 1)
-    (in_bom yes) (on_board yes) (dnp no) (fields_autoplaced)
-    (property "Reference" "#PWR058" (at 266.065 64.77 0)
-      (effects (font (size 1.27 1.27)) hide)
-    )
-    (property "Value" "+3.3V" (at 266.065 55.88 0)
-      (effects (font (size 1.27 1.27)))
-    )
-    (property "Footprint" "" (at 266.065 60.96 0)
-      (effects (font (size 1.27 1.27)) hide)
-    )
-    (property "Datasheet" "" (at 266.065 60.96 0)
-      (effects (font (size 1.27 1.27)) hide)
-    )
+  (symbol (lib_id "power:+3.3V") (at 266.7 78.105 0) (unit 1)
+    (in_bom yes) (on_board yes) (dnp no) (fields_autoplaced)
+    (property "Reference" "#PWR058" (at 266.7 81.915 0)
+      (effects (font (size 1.27 1.27)) hide)
+    )
+    (property "Value" "+3.3V" (at 266.7 73.025 0)
+      (effects (font (size 1.27 1.27)))
+    )
+    (property "Footprint" "" (at 266.7 78.105 0)
+      (effects (font (size 1.27 1.27)) hide)
+    )
+    (property "Datasheet" "" (at 266.7 78.105 0)
+      (effects (font (size 1.27 1.27)) hide)
+    )

Commit message: Update Control.kicad_sch
Connections:
- net +3V3 is gone; now on net +3.3V: C10.1, C11.1, C12.1, C13.1, C14.1, C15.1, C16.1, C5.1, C9.1, R2.2, U1.1 (IOVDD), U1.10 (IOVDD), U1.22 (IOVDD), U1.33 (IOVDD), U1.42 (IOVDD), U1.43 (ADC_AVDD), U1.44 (VREG_IN), U1.48 (USB_VDD), U1.49 (IOVDD), U2.8 (VCC)
Changed lines of the file:
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@@
+    (stroke (width 0) (type default))
+  )
+  (wire (pts (xy 125.095 28.575) (xy 133.985 28.575))
     (stroke (width 0) (type default))
   )
@@
     (stroke (width 0) (type default))
   )
-  (wire (pts (xy 46.355 60.96) (xy 46.355 62.865))
-    (stroke (width 0) (type default))
-  )
   (wire (pts (xy 264.16 88.265) (xy 264.16 116.205))
     (stroke (width 0) (type default))
@@
     (stroke (width 0) (type default))
   )
+  (wire (pts (xy 46.355 59.69) (xy 46.355 62.865))
+    (stroke (width 0) (type default))
+  )
   (wire (pts (xy 125.095 35.56) (xy 125.095 47.625))
     (stroke (width 0) (type default))
@@
     (stroke (width 0) (type default))
   )
-  (wire (pts (xy 125.095 31.115) (xy 125.095 35.56))
+  (wire (pts (xy 125.095 28.575) (xy 125.095 35.56))
     (stroke (width 0) (type default))
   )
@@
         (path "/c4c3980b-c8c0-435e-abdc-bbed2349d7ac/2f899246-8d98-4f9c-b4c6-8497c11eb038"
           (reference "R42") (unit 1)
-        )
-      )
-    )
-  )
-  (symbol (lib_id "power:+3V3") (at 125.095 31.115 0) (unit 1)
-    (in_bom yes) (on_board yes) (dnp no) (fields_autoplaced)
-    (property "Reference" "#PWR05" (at 125.095 34.925 0)
-      (effects (font (size 1.27 1.27)) hide)
-    )
-    (property "Value" "+3V3" (at 125.095 26.035 0)
-      (effects (font (size 1.27 1.27)))
-    )
-    (property "Footprint" "" (at 125.095 31.115 0)
-      (effects (font (size 1.27 1.27)) hide)
-    )
-    (property "Datasheet" "" (at 125.095 31.115 0)
-      (effects (font (size 1.27 1.27)) hide)
-    )
-    (pin "1")
-    (instances
-      (project "FufuS24"
-        (path "/c4c3980b-c8c0-435e-abdc-bbed2349d7ac/2f899246-8d98-4f9c-b4c6-8497c11eb038"
-          (reference "#PWR05") (unit 1)
         )
       )
@@
     )
   )
+  (symbol (lib_id "power:+3.3V") (at 46.355 59.69 0) (unit 1)
+    (in_bom yes) (on_board yes) (dnp no) (fields_autoplaced)
+    (property "Reference" "#PWR05" (at 46.355 63.5 0)
+      (effects (font (size 1.27 1.27)) hide)
+    )
+    (property "Value" "+3.3V" (at 46.355 54.61 0)
+      (effects (font (size 1.27 1.27)))
+    )
+    (property "Footprint" "" (at 46.355 59.69 0)
+      (effects (font (size 1.27 1.27)) hide)
+    )
+    (property "Datasheet" "" (at 46.355 59.69 0)
+      (effects (font (size 1.27 1.27)) hide)
+    )
+    (pin "1")
+    (instances
+      (project "FufuS24"
+        (path "/c4c3980b-c8c0-435e-abdc-bbed2349d7ac/2f899246-8d98-4f9c-b4c6-8497c11eb038"
+          (reference "#PWR05") (unit 1)
+        )
+      )
+    )
+  )
   (symbol (lib_id "Device:C") (at 91.44 39.37 0) (unit 1)
     (in_bom yes) (on_board yes) (dnp no) (fields_autoplaced)
@@
         (path "/c4c3980b-c8c0-435e-abdc-bbed2349d7ac/2f899246-8d98-4f9c-b4c6-8497c11eb038"
           (reference "C6") (unit 1)
+        )
+      )
+    )
+  )
+  (symbol (lib_id "power:+3.3V") (at 133.985 28.575 0) (unit 1)
+    (in_bom yes) (on_board yes) (dnp no) (fields_autoplaced)
+    (property "Reference" "#PWR053" (at 133.985 32.385 0)
+      (effects (font (size 1.27 1.27)) hide)
+    )
+    (property "Value" "+3.3V" (at 133.985 23.495 0)
+      (effects (font (size 1.27 1.27)))
+    )
+    (property "Footprint" "" (at 133.985 28.575 0)
+      (effects (font (size 1.27 1.27)) hide)
+    )
+    (property "Datasheet" "" (at 133.985 28.575 0)
+      (effects (font (size 1.27 1.27)) hide)
+    )
+    (pin "1")
+    (instances
+      (project "FufuS24"
+        (path "/c4c3980b-c8c0-435e-abdc-bbed2349d7ac/2f899246-8d98-4f9c-b4c6-8497c11eb038"
+          (reference "#PWR053") (unit 1)
         )
       )
@@
         )
       )
-    )
-  )
-  (symbol (lib_id "power:+3V3") (at 46.355 60.96 0) (unit 1)
-    (in_bom yes) (on_board yes) (dnp no) (fields_autoplaced)
-    (property "Reference" "#PWR010" (at 46.355 64.77 0)
-      (effects (font (size 1.27 1.27)) hide)
-    )
-    (property "Value" "+3V3" (at 46.355 55.88 0)
-      (effects (font (size 1.27 1.27)))
-    )
-    (property "Footprint" "" (at 46.355 60.96 0)
-      (effects (font (size 1.27 1.27)) hide)
-    )
-    (property "Datasheet" "" (at 46.355 60.96 0)
-      (effects (font (size 1.27 1.27)) hide)
-    )
-    (pin "1")
-    (instances
-      (project "FufuS24"
-        (path "/c4c3980b-c8c0-435e-abdc-bbed2349d7ac/2f899246-8d98-4f9c-b4c6-8497c11eb038"
-          (reference "#PWR010") (unit 1)
-        )
-      )

Commit message: if you're reading this aaaaaaa
Parts:
- C11, C12, C13, C14, C15, C16, C6, C7, C9: footprint footprints:CAPC2012X94N -> footprints:WCAP-CSGP_885012206026
Changed lines of the file:
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@@
       (effects (font (size 1.27 1.27)) (justify left))
     )
-    (property "Footprint" "footprints:CAPC2012X94N" (at 157.8102 43.18 0)
+    (property "Footprint" "footprints:WCAP-CSGP_885012206026" (at 157.8102 43.18 0)
       (effects (font (size 1.27 1.27)) hide)
     )
@@
       (effects (font (size 1.27 1.27)) (justify left))
     )
-    (property "Footprint" "footprints:CAPC2012X94N" (at 103.8352 43.18 0)
+    (property "Footprint" "footprints:WCAP-CSGP_885012206026" (at 103.8352 43.18 0)
       (effects (font (size 1.27 1.27)) hide)
     )
@@
       (effects (font (size 1.27 1.27)) (justify left))
     )
-    (property "Footprint" "footprints:CAPC2012X94N" (at 203.5302 43.18 0)
+    (property "Footprint" "footprints:WCAP-CSGP_885012206026" (at 203.5302 43.18 0)
       (effects (font (size 1.27 1.27)) hide)
     )
@@
       (effects (font (size 1.27 1.27)) (justify left))
     )
-    (property "Footprint" "footprints:CAPC2012X94N" (at 169.2402 43.18 0)
+    (property "Footprint" "footprints:WCAP-CSGP_885012206026" (at 169.2402 43.18 0)
       (effects (font (size 1.27 1.27)) hide)
     )
@@
       (effects (font (size 1.27 1.27)) (justify left))
     )
-    (property "Footprint" "footprints:CAPC2012X94N" (at 180.6702 43.18 0)
+    (property "Footprint" "footprints:WCAP-CSGP_885012206026" (at 180.6702 43.18 0)
       (effects (font (size 1.27 1.27)) hide)
     )
@@
       (effects (font (size 1.27 1.27)) (justify left))
     )
-    (property "Footprint" "footprints:CAPC2012X94N" (at 92.4052 43.18 0)
+    (property "Footprint" "footprints:WCAP-CSGP_885012206026" (at 92.4052 43.18 0)
       (effects (font (size 1.27 1.27)) hide)
     )
@@
       (effects (font (size 1.27 1.27)) (justify left))
     )
-    (property "Footprint" "footprints:CAPC2012X94N" (at 192.1002 43.18 0)
+    (property "Footprint" "footprints:WCAP-CSGP_885012206026" (at 192.1002 43.18 0)
       (effects (font (size 1.27 1.27)) hide)
     )
@@
       (effects (font (size 1.27 1.27)) (justify left))
     )
-    (property "Footprint" "footprints:CAPC2012X94N" (at 134.9502 43.18 0)
+    (property "Footprint" "footprints:WCAP-CSGP_885012206026" (at 134.9502 43.18 0)
       (effects (font (size 1.27 1.27)) hide)
     )
@@
       (effects (font (size 1.27 1.27)) (justify left))
     )
-    (property "Footprint" "footprints:CAPC2012X94N" (at 146.3802 43.18 0)
+    (property "Footprint" "footprints:WCAP-CSGP_885012206026" (at 146.3802 43.18 0)
       (effects (font (size 1.27 1.27)) hide)
     )
@@
       (effects (font (size 1.27 1.27)) (justify left top) hide)
     )
+    (pin "1")
+    (pin "10")
     (pin "11")
+    (pin "12")
+    (pin "13")
+    (pin "14")
+    (pin "15")
+    (pin "16")
+    (pin "17")
+    (pin "18")
+    (pin "19")
+    (pin "2")
+    (pin "20")
+    (pin "21")
+    (pin "22")
+    (pin "23")
     (pin "24")
     (pin "3")
@@
     (pin "7")
     (pin "8")
-    (pin "12")
-    (pin "2")
-    (pin "20")
-    (pin "21")
-    (pin "22")
-    (pin "23")
-    (pin "14")
-    (pin "15")
-    (pin "16")
-    (pin "17")
-    (pin "18")
-    (pin "19")
-    (pin "1")
     (pin "9")
-    (pin "10")
-    (pin "13")
-    (instances
-      (project "FufuS24"
+    (instances
+      (project "FufuS24"
