File: production/ecad/FufuS24/Motor.kicad_sch (KiCad schematic)
At the start: 12 parts, among them J10 Conn_01x02, J11 Conn_01x02, J12 Conn_01x02, J13 Conn_01x03_Socket, J5 Conn_01x02, J6 Conn_01x02, J7 Conn_01x03_Socket, J8 Conn_01x02, J9 Conn_01x02

Commit message: efan 3
Parts:
- J5, J6, J7: footprint (none) -> footprints:CONN2_710002_WRE
Changed lines of the file:
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@@
       (effects (font (size 1.27 1.27)))
     )
-    (property "Footprint" "" (at 32.385 60.325 0)
+    (property "Footprint" "footprints:CONN2_710002_WRE" (at 32.385 60.325 0)
       (effects (font (size 1.27 1.27)) hide)
     )
@@
       (effects (font (size 1.27 1.27)))
     )
-    (property "Footprint" "" (at 31.115 83.82 0)
+    (property "Footprint" "footprints:CONN2_710002_WRE" (at 31.115 83.82 0)
       (effects (font (size 1.27 1.27)) hide)
     )
@@
       (effects (font (size 1.27 1.27)))
     )
-    (property "Footprint" "" (at 32.385 38.1 0)
-      (effects (font (size 1.27 1.27)) hide)
-    )
+    (property "Footprint" "footprints:CONN2_710002_WRE" (at 32.385 38.1 0)
+      (effects (font (size 1.27 1.27)) hide)
+    )

Commit message: efan 5
Parts:
- J10, J11, J12, J8, J9: footprint (none) -> footprints:CON_5025840270_MOL
- TP6, TP7, TP8: footprint TestPoint:TestPoint_Pad_2.0x2.0mm -> footprints:TP_5014
Changed lines of the file:
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@@
       (effects (font (size 1.27 1.27)))
     )
-    (property "Footprint" "" (at 32.385 104.775 0)
+    (property "Footprint" "footprints:CON_5025840270_MOL" (at 32.385 104.775 0)
       (effects (font (size 1.27 1.27)) hide)
     )
@@
       (effects (font (size 1.27 1.27)) (justify left))
     )
-    (property "Footprint" "TestPoint:TestPoint_Pad_2.0x2.0mm" (at 111.76 54.61 0)
+    (property "Footprint" "footprints:TP_5014" (at 111.76 54.61 0)
       (effects (font (size 1.27 1.27)) hide)
     )
@@
       (effects (font (size 1.27 1.27)))
     )
-    (property "Footprint" "" (at 32.385 151.13 0)
+    (property "Footprint" "footprints:CON_5025840270_MOL" (at 32.385 151.13 0)
       (effects (font (size 1.27 1.27)) hide)
     )
@@
       (effects (font (size 1.27 1.27)))
     )
-    (property "Footprint" "" (at 32.385 132.715 0)
+    (property "Footprint" "footprints:CON_5025840270_MOL" (at 32.385 132.715 0)
       (effects (font (size 1.27 1.27)) hide)
     )
@@
       (effects (font (size 1.27 1.27)) (justify left))
     )
-    (property "Footprint" "TestPoint:TestPoint_Pad_2.0x2.0mm" (at 109.855 43.815 0)
+    (property "Footprint" "footprints:TP_5014" (at 109.855 43.815 0)
       (effects (font (size 1.27 1.27)) hide)
     )
@@
       (effects (font (size 1.27 1.27)))
     )
-    (property "Footprint" "" (at 32.385 110.49 0)
+    (property "Footprint" "footprints:CON_5025840270_MOL" (at 32.385 110.49 0)
       (effects (font (size 1.27 1.27)) hide)
     )
@@
       (effects (font (size 1.27 1.27)) (justify right))
     )
-    (property "Footprint" "TestPoint:TestPoint_Pad_2.0x2.0mm" (at 99.695 55.88 0)
+    (property "Footprint" "footprints:TP_5014" (at 99.695 55.88 0)
       (effects (font (size 1.27 1.27)) hide)
     )
@@
       (effects (font (size 1.27 1.27)))
     )
-    (property "Footprint" "" (at 32.385 127 0)
-      (effects (font (size 1.27 1.27)) hide)
-    )
+    (property "Footprint" "footprints:CON_5025840270_MOL" (at 32.385 127 0)
+      (effects (font (size 1.27 1.27)) hide)
+    )

Commit message: goose
Parts:
- removed J11, J8, J9: Conn_01x02, footprints:CON_5025840270_MOL, symbol Connector_Generic:Conn_01x02
- removed J5, J6: Conn_01x02, footprints:CONN2_710002_WRE, symbol Connector_Generic:Conn_01x02
- removed J7: Conn_01x03_Socket, footprints:CONN2_710002_WRE, symbol Connector:Conn_01x03_Socket
- added U12: Pololu_DRV8711_Motor_Driver, symbol POLOLU_35v4:Pololu_DRV8711_Motor_Driver
- J10, J12: footprint footprints:CON_5025840270_MOL -> (none)
- TP6, TP7, TP8: footprint footprints:TP_5014 -> TestPoint:TestPoint_Pad_2.0x2.0mm
Connections:
- net +48V: now also U12.1 (Vin), U12.21 (VM)
- net +5V: now also U12.19 (ICREF), U12.20 (V5(OUT))
- net GNDREF: now also U12.22 (GND)
- net Motor_BIN1: now also U12.9 (BIN1)
- net Motor_BIN2: now also U12.8 (BIN2)
- net Motor_DIR: now also U12.17 (DIR)
- net Motor_SPI1_CLK: now also U12.14 (SCLK)
- net Motor_SPI1_CSn: now also U12.13 (SCS)
- net Motor_Step: now also U12.18 (STEP)
Other:
- note removed: "48V Motor ctrl pwr input"
- note removed: "5V Logic pwr"
- note removed: "BIN1"
- note removed: "BIN2"
- note removed: "Current limited power...perchance"
- note removed: "DIR"
- note removed: "GND"
- note removed: "IOREF"
- note removed: "PWM Ctrl"
- note removed: "SCLK"
- note removed: "SCS"
- note removed: "STEP"
- note removed: "V5_OUT"
- note removed: "VIN"
- note removed: "VM"

Commit message: Update Motor.kicad_sch
Parts:
- added J5: 691137710004, 691137710004:WURTH_691137710004, symbol PWR_4POS:691137710004
Changed lines of the file:
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@@
+    )
+  )
+  (symbol (lib_id "PWR_4POS:691137710004") (at 33.655 45.72 0) (unit 1)
+    (in_bom yes) (on_board yes) (dnp no) (fields_autoplaced)
+    (property "Reference" "J5" (at 40.64 45.72 0)
+      (effects (font (size 1.27 1.27)) (justify left))
+    )
+    (property "Value" "691137710004" (at 40.64 48.26 0)
+      (effects (font (size 1.27 1.27)) (justify left))
+    )
+    (property "Footprint" "691137710004:WURTH_691137710004" (at 33.655 45.72 0)
+      (effects (font (size 1.27 1.27)) (justify bottom) hide)
+    )
+    (property "Datasheet" "" (at 33.655 45.72 0)
+      (effects (font (size 1.27 1.27)) hide)
+    )
+    (property "MF" "Wurth Electronics" (at 33.655 45.72 0)
+      (effects (font (size 1.27 1.27)) (justify bottom) hide)
+    )
+    (property "MAXIMUM_PACKAGE_HEIGHT" "11.6mm" (at 33.655 45.72 0)
+      (effects (font (size 1.27 1.27)) (justify bottom) hide)
+    )
+    (property "Package" "None" (at 33.655 45.72 0)
+      (effects (font (size 1.27 1.27)) (justify bottom) hide)
+    )
+    (property "Price" "None" (at 33.655 45.72 0)
+      (effects (font (size 1.27 1.27)) (justify bottom) hide)
+    )
+    (property "Check_prices" "https://www.snapeda.com/parts/691137710004/Wurth+Electronics+Inc./view-part/?ref=eda" (at 33.655 45.72 0)
+      (effects (font (size 1.27 1.27)) (justify bottom) hide)
+    )
+    (property "STANDARD" "Manufacturer Recommendations" (at 33.655 45.72 0)
+      (effects (font (size 1.27 1.27)) (justify bottom) hide)
+    )
+    (property "PARTREV" "001" (at 33.655 45.72 0)
+      (effects (font (size 1.27 1.27)) (justify bottom) hide)
+    )
+    (property "SnapEDA_Link" "https://www.snapeda.com/parts/691137710004/Wurth+Electronics+Inc./view-part/?ref=snap" (at 33.655 45.72 0)
+      (effects (font (size 1.27 1.27)) (justify bottom) hide)
+    )
+    (property "MP" "691137710004" (at 33.655 45.72 0)
+      (effects (font (size 1.27 1.27)) (justify bottom) hide)
+    )
+    (property "Purchase-URL" "https://www.snapeda.com/api/url_track_click_mouser/?unipart_id=2900223&manufacturer=Wurth Electronics&part_name=691137710004&search_term=691137710004" (at 33.655 45.72 0)
+      (effects (font (size 1.27 1.27)) (justify bottom) hide)
+    )
+    (property "Description" "\n4 Position Wire to Board Terminal Block Horizontal with Board 0.197 (5.00mm) Through Hole\n" (at 33.655 45.72 0)
+      (effects (font (size 1.27 1.27)) (justify bottom) hide)
+    )
+    (property "Availability" "In Stock" (at 33.655 45.72 0)
+      (effects (font (size 1.27 1.27)) (justify bottom) hide)
+    )
+    (property "MANUFACTURER" "WURTH ELEKTRONIK" (at 33.655 45.72 0)
+      (effects (font (size 1.27 1.27)) (justify bottom) hide)
+    )
+    (pin "1")
+    (pin "2")
+    (pin "3")
+    (pin "4")
+    (instances
+      (project "FufuS24"
+        (path "/c4c3980b-c8c0-435e-abdc-bbed2349d7ac/67add6e2-1584-4801-9b59-67cf5082dcca"
+          (reference "J5") (unit 1)
+        )
+      )
     )
   )

Commit message: Efan 6
Parts:
- TP6, TP7, TP8: footprint TestPoint:TestPoint_Pad_2.0x2.0mm -> footprints:TP_5014
Changed lines of the file:
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@@
       (effects (font (size 1.27 1.27)) (justify left))
     )
-    (property "Footprint" "TestPoint:TestPoint_Pad_2.0x2.0mm" (at 111.76 54.61 0)
+    (property "Footprint" "footprints:TP_5014" (at 111.76 54.61 0)
       (effects (font (size 1.27 1.27)) hide)
     )
@@
       (effects (font (size 1.27 1.27)) (justify left))
     )
-    (property "Footprint" "TestPoint:TestPoint_Pad_2.0x2.0mm" (at 109.855 43.815 0)
+    (property "Footprint" "footprints:TP_5014" (at 109.855 43.815 0)
       (effects (font (size 1.27 1.27)) hide)
     )
@@
   (symbol (lib_id "power:+48V") (at 118.745 83.82 90) (unit 1)
     (in_bom yes) (on_board yes) (dnp no)
-    (property "Reference" "#PWR053" (at 122.555 83.82 0)
+    (property "Reference" "#PWR0101" (at 122.555 83.82 0)
       (effects (font (size 1.27 1.27)) hide)
     )
@@
       (project "FufuS24"
         (path "/c4c3980b-c8c0-435e-abdc-bbed2349d7ac/67add6e2-1584-4801-9b59-67cf5082dcca"
-          (reference "#PWR053") (unit 1)
+          (reference "#PWR0101") (unit 1)
         )
       )
@@
       (effects (font (size 1.27 1.27)) (justify right))
     )
-    (property "Footprint" "TestPoint:TestPoint_Pad_2.0x2.0mm" (at 99.695 55.88 0)
-      (effects (font (size 1.27 1.27)) hide)
-    )
+    (property "Footprint" "footprints:TP_5014" (at 99.695 55.88 0)
+      (effects (font (size 1.27 1.27)) hide)
+    )

Commit message: efan 7
Parts:
- J10, J12: footprint (none) -> footprints:CON_5025840270_MOL
- U12: footprint (none) -> footprints:POLOLU_36v4
Changed lines of the file:
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@@
       (effects (font (size 1.27 1.27)))
     )
-    (property "Footprint" "" (at 32.385 151.13 0)
+    (property "Footprint" "footprints:CON_5025840270_MOL" (at 32.385 151.13 0)
       (effects (font (size 1.27 1.27)) hide)
     )
@@
       (effects (font (size 1.524 1.524)))
     )
-    (property "Footprint" "" (at 119.38 78.74 0)
+    (property "Footprint" "footprints:POLOLU_36v4" (at 119.38 78.74 0)
       (effects (font (size 1.27 1.27) italic) hide)
     )
@@
       (effects (font (size 1.27 1.27)))
     )
-    (property "Footprint" "" (at 32.385 127 0)
-      (effects (font (size 1.27 1.27)) hide)
-    )
+    (property "Footprint" "footprints:CON_5025840270_MOL" (at 32.385 127 0)
+      (effects (font (size 1.27 1.27)) hide)
+    )
