File: production/ecad/FufuS24/Water_Dispensing.kicad_sch (KiCad schematic)
At the start: 2 parts, among them Q1 DMG2302UK-7

Commit message: efan 3
Parts:
- R20: footprint (none) -> footprints:RESC2012X60N
Changed lines of the file:
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@@
       (effects (font (size 1.27 1.27)) (justify left))
     )
-    (property "Footprint" "" (at 68.326 45.974 90)
+    (property "Footprint" "footprints:RESC2012X60N" (at 68.326 45.974 90)
       (effects (font (size 1.27 1.27)) hide)
     )

Commit message: goose
Parts:
- R20: footprint footprints:RESC2012X60N -> (none)
Changed lines of the file:
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@@
       (effects (font (size 1.27 1.27)) (justify left))
     )
-    (property "Footprint" "footprints:RESC2012X60N" (at 68.326 45.974 90)
+    (property "Footprint" "" (at 68.326 45.974 90)
       (effects (font (size 1.27 1.27)) hide)
     )

Commit message: Efan 6
Parts:
- R20: footprint (none) -> footprints:RESC2012X60N
Changed lines of the file:
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@@
       (effects (font (size 1.27 1.27)) (justify left))
     )
-    (property "Footprint" "" (at 68.326 45.974 90)
+    (property "Footprint" "footprints:RESC2012X60N" (at 68.326 45.974 90)
       (effects (font (size 1.27 1.27)) hide)
     )

Commit message: eLISE MOTOR FIXED
Parts:
- R20: footprint footprints:RESC2012X60N -> (none)
Changed lines of the file:
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@@
       (effects (font (size 1.27 1.27)) (justify left))
     )
-    (property "Footprint" "footprints:RESC2012X60N" (at 68.326 45.974 90)
+    (property "Footprint" "" (at 68.326 45.974 90)
       (effects (font (size 1.27 1.27)) hide)
     )
