File: production/ecad/FufuS24/Induction_Heating.kicad_sch (KiCad schematic)
At the start: 17 parts, among them J1 Conn_01x02, J14 691137710002, M1 MLX90614ESF-AAA-000-TU

Commit message: goose
Parts:
- removed J14: 691137710002, footprints:CONN2_710002_WRE, symbol 2024-03-03_19-32-21:691137710002
- C17: footprint footprints:CAPC2012X94N -> footprints:U1-E_NCH
- C17: renamed from C49; footprint footprints:CAPC2012X94N -> 8600footprint:CAP_WCAP-ATG5_05.0X11.0_WRE
- C18: footprint footprints:CAPC2012X94N -> 8600footprint:CAP_WCAP-ATG5_05.0X11.0_WRE
- C4: footprint footprints:CAPC2012X94N -> KiCad:ECQUAAF335LD
- J1: footprint footprints:CON_5025840270_MOL -> B2B-XH-A_LF__SN_:JST_B2B-XH-A_LF__SN_
- R11, R6, R7, R8: footprint footprints:RESC2012X60N -> (none)
- R9: footprint footprints:RESC2012X60N -> SQPfootprints:RES_SQP500_22X9P5_YAG
- TP9: footprint footprints:TP_5014 -> TestPoint:TestPoint_Pad_2.0x2.0mm
Changed lines of the file:
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@@
-    (stroke (width 0) (type default))
-  )
-  (wire (pts (xy 41.91 41.275) (xy 47.625 41.275))
     (stroke (width 0) (type default))
   )
@@
     (stroke (width 0) (type default))
   )
-  (wire (pts (xy 41.91 38.735) (xy 47.625 38.735))
-    (stroke (width 0) (type default))
-  )
   (wire (pts (xy 49.53 147.32) (xy 55.88 147.32))
     (stroke (width 0) (type default))
@@
   (label "VSS" (at 76.2 147.32 0) (fields_autoplaced)
     (effects (font (size 1.27 1.27)) (justify left bottom))
-  )
-  (global_label "Temp_Light_Neg" (shape input) (at 41.91 41.275 180) (fields_autoplaced)
-    (effects (font (size 1.27 1.27)) (justify right))
-    (property "Intersheetrefs" "${INTERSHEET_REFS}" (at 23.8664 41.275 0)
-      (effects (font (size 1.27 1.27)) (justify right) hide)
-    )
   )
   (global_label "Heat_PWM1" (shape input) (at 26.67 138.43 180) (fields_autoplaced)
@@
     )
   )
-  (global_label "Temp_Light_Pos" (shape input) (at 41.91 38.735 180) (fields_autoplaced)
-    (effects (font (size 1.27 1.27)) (justify right))
-    (property "Intersheetrefs" "${INTERSHEET_REFS}" (at 23.9874 38.735 0)
-      (effects (font (size 1.27 1.27)) (justify right) hide)
-    )
-  )
   (global_label "I2C0_SCL" (shape input) (at 265.43 80.01 0) (fields_autoplaced)
     (effects (font (size 1.27 1.27)) (justify left))
@@
       (effects (font (size 1.27 1.27)) hide)
     )
+    (pin "1")
     (pin "2")
     (pin "3")
-    (pin "1")
     (instances
       (project "FufuS24"
         (path "/c4c3980b-c8c0-435e-abdc-bbed2349d7ac/57fb5dcd-e779-40d3-8741-57c7eee1ca58"
           (reference "U9") (unit 1)
-        )
-      )
-    )
-  )
-  (symbol (lib_id "2024-03-03_19-32-21:691137710002") (at 47.625 38.735 0) (unit 1)
-    (in_bom yes) (on_board yes) (dnp no) (fields_autoplaced)
-    (property "Reference" "J14" (at 62.23 38.735 0)
-      (effects (font (size 1.524 1.524)) (justify left))
-    )
-    (property "Value" "691137710002" (at 62.23 41.275 0)
-      (effects (font (size 1.524 1.524)) (justify left))
-    )
-    (property "Footprint" "footprints:CONN2_710002_WRE" (at 47.625 38.735 0)
-      (effects (font (size 1.27 1.27) italic) hide)
-    )
-    (property "Datasheet" "691137710002" (at 47.625 38.735 0)
-      (effects (font (size 1.27 1.27) italic) hide)
-    )
-    (pin "1")
-    (pin "2")
-    (instances
-      (project "FufuS24"
-        (path "/c4c3980b-c8c0-435e-abdc-bbed2349d7ac/57fb5dcd-e779-40d3-8741-57c7eee1ca58"
-          (reference "J14") (unit 1)
         )
       )
@@
       (effects (font (size 1.27 1.27)))
     )
-    (property "Footprint" "footprints:RESC2012X60N" (at 122.174 161.036 90)
+    (property "Footprint" "" (at 122.174 161.036 90)
       (effects (font (size 1.27 1.27)) hide)
     )
@@
       (effects (font (size 1.27 1.27)) (justify left))
     )
-    (property "Footprint" "footprints:TP_5014" (at 135.89 165.1 0)
+    (property "Footprint" "TestPoint:TestPoint_Pad_2.0x2.0mm" (at 135.89 165.1 0)
       (effects (font (size 1.27 1.27)) hide)
     )
@@
       (effects (font (size 1.27 1.27)) (justify left))
     )
-    (property "Footprint" "footprints:CAPC2012X94N" (at 83.82 118.11 0)
+    (property "Footprint" "footprints:U1-E_NCH" (at 83.82 118.11 0)
       (effects (font (size 1.27 1.27) italic) hide)
     )
@@
       (effects (font (size 1.27 1.27)) (justify left))
     )
-    (property "Footprint" "footprints:RESC2012X60N" (at 106.68 160.02 0)
+    (property "Footprint" "SQPfootprints:RES_SQP500_22X9P5_YAG" (at 106.68 160.02 0)
       (effects (font (size 1.27 1.27) italic) hide)
     )
@@
       (effects (font (size 1.27 1.27)))
     )
-    (property "Footprint" "footprints:CON_5025840270_MOL" (at 123.19 104.14 0)
+    (property "Footprint" "B2B-XH-A_LF__SN_:JST_B2B-XH-A_LF__SN_" (at 123.19 104.14 0)
       (effects (font (size 1.27 1.27)) hide)
     )
@@
       (effects (font (size 1.27 1.27)) (justify bottom) hide)
     )
+    (pin "1")
+    (pin "2")
+    (pin "3")
     (pin "4")
-    (pin "3")
-    (pin "2")
-    (pin "1")
     (instances
       (project "FufuS24"
@@
   (symbol (lib_id "2023-11-09_20-51-41:860020772001") (at 132.08 165.1 270) (unit 1)
     (in_bom yes) (on_board yes) (dnp no) (fields_autoplaced)
-    (property "Reference" "C49" (at 135.89 167.64 90)
+    (property "Reference" "C17" (at 135.89 167.64 90)
       (effects (font (size 1.27 1.27)) (justify left))
     )
@@
       (effects (font (size 1.27 1.27)) (justify left))
     )
-    (property "Footprint" "footprints:CAPC2012X94N" (at 132.08 165.1 0)
+    (property "Footprint" "8600footprint:CAP_WCAP-ATG5_05.0X11.0_WRE" (at 132.08 165.1 0)
       (effects (font (size 1.27 1.27) italic) hide)
     )
@@
       (project "FufuS24"
         (path "/c4c3980b-c8c0-435e-abdc-bbed2349d7ac/57fb5dcd-e779-40d3-8741-57c7eee1ca58"
-          (reference "C49") (unit 1)
+          (reference "C17") (unit 1)
         )
       )
@@
       (effects (font (size 1.27 1.27)))
     )
-    (property "Footprint" "footprints:RESC2012X60N" (at 39.624 137.414 90)
+    (property "Footprint" "" (at 39.624 137.414 90)
       (effects (font (size 1.27 1.27)) hide)
     )
@@
       (effects (font (size 1.27 1.27)))
     )
-    (property "Footprint" "footprints:RESC2012X60N" (at 87.249 137.414 90)
+    (property "Footprint" "" (at 87.249 137.414 90)
       (effects (font (size 1.27 1.27)) hide)
     )
@@
       (effects (font (size 1.27 1.27)))
     )
-    (property "Footprint" "footprints:CAPC2012X94N" (at 149.86 178.74 0)
+    (property "Footprint" "KiCad:ECQUAAF335LD" (at 149.86 178.74 0)
       (effects (font (size 1.27 1.27)) (justify left top) hide)
     )
@@
       (effects (font (size 1.27 1.27)) (justify left))
     )
-    (property "Footprint" "footprints:CAPC2012X94N" (at 257.81 95.25 0)
+    (property "Footprint" "8600footprint:CAP_WCAP-ATG5_05.0X11.0_WRE" (at 257.81 95.25 0)
       (effects (font (size 1.27 1.27) italic) hide)
     )
@@
       (effects (font (size 1.27 1.27)) (justify right))
     )
-    (property "Footprint" "footprints:RESC2012X60N" (at 91.694 148.336 90)
+    (property "Footprint" "" (at 91.694 148.336 90)
       (effects (font (size 1.27 1.27)) hide)
     )
@@
       (effects (font (size 1.27 1.27)) hide)
     )
+    (pin "1")
+    (pin "2")
+    (pin "3")
+    (pin "4")
+    (pin "5")
     (pin "6")
-    (pin "5")
-    (pin "4")
+    (pin "7")
     (pin "8")
-    (pin "7")
-    (pin "1")
-    (pin "2")
-    (pin "3")
-    (instances
-      (project "FufuS24"
+    (instances
+      (project "FufuS24"

Commit message: Efan 6
Parts:
- C17: footprint footprints:U1-E_NCH -> footprints:CAPC2012X94N
- C18: footprint 8600footprint:CAP_WCAP-ATG5_05.0X11.0_WRE -> footprints:CAPC2012X94N
- C4: footprint KiCad:ECQUAAF335LD -> footprints:CAPC2012X94N
- C51: renamed from C17; footprint 8600footprint:CAP_WCAP-ATG5_05.0X11.0_WRE -> footprints:CAPC2012X94N
- R11, R6, R7, R8: footprint (none) -> footprints:RESC2012X60N
- R9: footprint SQPfootprints:RES_SQP500_22X9P5_YAG -> footprints:RESC2012X60N
- TP9: footprint TestPoint:TestPoint_Pad_2.0x2.0mm -> footprints:TP_5014
Changed lines of the file:
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@@
       (effects (font (size 1.27 1.27)))
     )
-    (property "Footprint" "" (at 122.174 161.036 90)
+    (property "Footprint" "footprints:RESC2012X60N" (at 122.174 161.036 90)
       (effects (font (size 1.27 1.27)) hide)
     )
@@
       (effects (font (size 1.27 1.27)) (justify left))
     )
-    (property "Footprint" "TestPoint:TestPoint_Pad_2.0x2.0mm" (at 135.89 165.1 0)
+    (property "Footprint" "footprints:TP_5014" (at 135.89 165.1 0)
       (effects (font (size 1.27 1.27)) hide)
     )
@@
       (effects (font (size 1.27 1.27)) (justify left))
     )
-    (property "Footprint" "footprints:U1-E_NCH" (at 83.82 118.11 0)
+    (property "Footprint" "footprints:CAPC2012X94N" (at 83.82 118.11 0)
       (effects (font (size 1.27 1.27) italic) hide)
     )
@@
       (effects (font (size 1.27 1.27)) (justify left))
     )
-    (property "Footprint" "SQPfootprints:RES_SQP500_22X9P5_YAG" (at 106.68 160.02 0)
+    (property "Footprint" "footprints:RESC2012X60N" (at 106.68 160.02 0)
       (effects (font (size 1.27 1.27) italic) hide)
     )
@@
   (symbol (lib_id "2023-11-09_20-51-41:860020772001") (at 132.08 165.1 270) (unit 1)
     (in_bom yes) (on_board yes) (dnp no) (fields_autoplaced)
-    (property "Reference" "C17" (at 135.89 167.64 90)
+    (property "Reference" "C51" (at 135.89 167.64 90)
       (effects (font (size 1.27 1.27)) (justify left))
     )
@@
       (effects (font (size 1.27 1.27)) (justify left))
     )
-    (property "Footprint" "8600footprint:CAP_WCAP-ATG5_05.0X11.0_WRE" (at 132.08 165.1 0)
+    (property "Footprint" "footprints:CAPC2012X94N" (at 132.08 165.1 0)
       (effects (font (size 1.27 1.27) italic) hide)
     )
@@
       (project "FufuS24"
         (path "/c4c3980b-c8c0-435e-abdc-bbed2349d7ac/57fb5dcd-e779-40d3-8741-57c7eee1ca58"
-          (reference "C17") (unit 1)
+          (reference "C51") (unit 1)
         )
       )
@@
       (effects (font (size 1.27 1.27)))
     )
-    (property "Footprint" "" (at 39.624 137.414 90)
+    (property "Footprint" "footprints:RESC2012X60N" (at 39.624 137.414 90)
       (effects (font (size 1.27 1.27)) hide)
     )
@@
       (effects (font (size 1.27 1.27)))
     )
-    (property "Footprint" "" (at 87.249 137.414 90)
+    (property "Footprint" "footprints:RESC2012X60N" (at 87.249 137.414 90)
       (effects (font (size 1.27 1.27)) hide)
     )
@@
       (effects (font (size 1.27 1.27)))
     )
-    (property "Footprint" "KiCad:ECQUAAF335LD" (at 149.86 178.74 0)
+    (property "Footprint" "footprints:CAPC2012X94N" (at 149.86 178.74 0)
       (effects (font (size 1.27 1.27)) (justify left top) hide)
     )
@@
       (effects (font (size 1.27 1.27)) (justify left))
     )
-    (property "Footprint" "8600footprint:CAP_WCAP-ATG5_05.0X11.0_WRE" (at 257.81 95.25 0)
+    (property "Footprint" "footprints:CAPC2012X94N" (at 257.81 95.25 0)
       (effects (font (size 1.27 1.27) italic) hide)
     )
@@
       (effects (font (size 1.27 1.27)) (justify right))
     )
-    (property "Footprint" "" (at 91.694 148.336 90)
-      (effects (font (size 1.27 1.27)) hide)
-    )
+    (property "Footprint" "footprints:RESC2012X60N" (at 91.694 148.336 90)
+      (effects (font (size 1.27 1.27)) hide)
+    )

Commit message: efan 7
Parts:
- J1: footprint B2B-XH-A_LF__SN_:JST_B2B-XH-A_LF__SN_ -> footprints:CONN2_710002_WRE
- L1: footprint INDPM:INDPM176169X700N -> footprints:INDPM120120X800N
Changed lines of the file:
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@@
       (effects (font (size 1.27 1.27)) (justify left))
     )
-    (property "Footprint" "INDPM:INDPM176169X700N" (at 35.255 78.74 0)
+    (property "Footprint" "footprints:INDPM120120X800N" (at 35.255 78.74 0)
       (effects (font (size 1.27 1.27)) (justify left top) hide)
     )
@@
       (effects (font (size 1.27 1.27)))
     )
-    (property "Footprint" "B2B-XH-A_LF__SN_:JST_B2B-XH-A_LF__SN_" (at 123.19 104.14 0)
+    (property "Footprint" "footprints:CONN2_710002_WRE" (at 123.19 104.14 0)
       (effects (font (size 1.27 1.27)) hide)
     )

Commit message: efan 8
Parts:
- M1: footprint MLX90614ESF-AAA-000-TU:TO254P942H425-4 -> footprints:IR_Sensor
Changed lines of the file:
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@@
       (effects (font (size 1.27 1.27)))
     )
-    (property "Footprint" "MLX90614ESF-AAA-000-TU:TO254P942H425-4" (at 220.98 95.25 0)
+    (property "Footprint" "footprints:IR_Sensor" (at 220.98 95.25 0)
       (effects (font (size 1.27 1.27)) (justify bottom) hide)
     )

Commit message: efan 9
Parts:
- added J6: 5025840270, CON_5025840270_MOL, symbol molex-2pos:5025840270
Connections:
- new net HOT_LED_NEG: J6.1
- new net HOT_LED_POS: J6.2
Changed lines of the file:
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@@
+    (stroke (width 0) (type default))
+  )
+  (wire (pts (xy 51.435 48.895) (xy 45.085 48.895))
     (stroke (width 0) (type default))
   )
@@
   )
   (wire (pts (xy 132.08 101.6) (xy 128.27 101.6))
+    (stroke (width 0) (type default))
+  )
+  (wire (pts (xy 51.435 46.355) (xy 45.085 46.355))
     (stroke (width 0) (type default))
   )
@@
     )
   )
+  (global_label "HOT_LED_POS" (shape input) (at 51.435 46.355 0) (fields_autoplaced)
+    (effects (font (size 1.27 1.27)) (justify left))
+    (property "Intersheetrefs" "${INTERSHEET_REFS}" (at 67.2411 46.355 0)
+      (effects (font (size 1.27 1.27)) (justify left) hide)
+    )
+  )
   (global_label "I2C0_SDA" (shape input) (at 265.43 76.2 0) (fields_autoplaced)
     (effects (font (size 1.27 1.27)) (justify left))
@@
     )
   )
+  (global_label "HOT_LED_NEG" (shape input) (at 51.435 48.895 0) (fields_autoplaced)
+    (effects (font (size 1.27 1.27)) (justify left))
+    (property "Intersheetrefs" "${INTERSHEET_REFS}" (at 67.1806 48.895 0)
+      (effects (font (size 1.27 1.27)) (justify left) hide)
+    )
+  )
   (global_label "I2C0_SCL" (shape input) (at 265.43 80.01 0) (fields_autoplaced)
     (effects (font (size 1.27 1.27)) (justify left))
@@
         )
       )
+    )
+  )
+  (symbol (lib_id "molex-2pos:5025840270") (at 45.085 48.895 180) (unit 1)
+    (in_bom yes) (on_board yes) (dnp no) (fields_autoplaced)
+    (property "Reference" "J6" (at 36.195 34.29 0)
+      (effects (font (size 1.524 1.524)))
+    )
+    (property "Value" "5025840270" (at 36.195 36.83 0)
+      (effects (font (size 1.524 1.524)))
+    )
+    (property "Footprint" "CON_5025840270_MOL" (at 45.085 48.895 0)
+      (effects (font (size 1.27 1.27) italic) hide)
+    )
+    (property "Datasheet" "5025840270" (at 45.085 48.895 0)
+      (effects (font (size 1.27 1.27) italic) hide)
+    )
+    (pin "4")
+    (pin "3")
+    (pin "2")
+    (pin "1")
+    (instances
+      (project "FufuS24"
+        (path "/c4c3980b-c8c0-435e-abdc-bbed2349d7ac/57fb5dcd-e779-40d3-8741-57c7eee1ca58"
+          (reference "J6") (unit 1)
+        )
+      )

Commit message: Footprints
Parts:
- J6: footprint CON_5025840270_MOL -> footprints:CON_5025840270_MOL
- U8, U9: footprint (none) -> footprints:TP_5014
Changed lines of the file:
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@@
       (effects (font (size 1.27 1.27)))
     )
-    (property "Footprint" "" (at 109.22 130.81 0)
+    (property "Footprint" "footprints:TP_5014" (at 109.22 130.81 0)
       (effects (font (size 1.27 1.27)) hide)
     )
@@
       (effects (font (size 1.524 1.524)))
     )
-    (property "Footprint" "CON_5025840270_MOL" (at 45.085 48.895 0)
+    (property "Footprint" "footprints:CON_5025840270_MOL" (at 45.085 48.895 0)
       (effects (font (size 1.27 1.27) italic) hide)
     )
@@
       (effects (font (size 1.27 1.27)))
     )
-    (property "Footprint" "" (at 60.96 132.08 0)
-      (effects (font (size 1.27 1.27)) hide)
-    )
+    (property "Footprint" "footprints:TP_5014" (at 60.96 132.08 0)
+      (effects (font (size 1.27 1.27)) hide)
+    )

Commit message: Final Foot Fetish
Parts:
- C35: footprint ECWF6754HL:CAPRR2500W80L2800T1330H1990 -> footprints:CAPC2012X94N
Changed lines of the file:
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@@
       (effects (font (size 1.27 1.27)) (justify right))
     )
-    (property "Footprint" "ECWF6754HL:CAPRR2500W80L2800T1330H1990" (at 140.97 102.87 0)
+    (property "Footprint" "footprints:CAPC2012X94N" (at 140.97 102.87 0)
       (effects (font (size 1.27 1.27)) (justify bottom) hide)
     )

Commit message: efan finals before laying out
Parts:
- removed TP9: TestPoint, footprints:TP_5014, symbol Connector:TestPoint
- added TP9: 5014, footprints:TP_5014, symbol 5014:5014
- U8: footprint footprints:TP_5014 -> footprints:FOD3150_footprint
- U9: footprint footprints:TP_5014 -> footprints:IRFB4610PBF
Connections:
- net at C51.1, R11.2: now also TP9.TP
Changed lines of the file:
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@@
       (effects (font (size 1.27 1.27)))
     )
-    (property "Footprint" "footprints:TP_5014" (at 109.22 130.81 0)
+    (property "Footprint" "footprints:IRFB4610PBF" (at 109.22 130.81 0)
       (effects (font (size 1.27 1.27)) hide)
     )
@@
     )
   )
-  (symbol (lib_id "Connector:TestPoint") (at 135.89 160.02 270) (unit 1)
-    (in_bom yes) (on_board yes) (dnp no) (fields_autoplaced)
-    (property "Reference" "TP9" (at 140.97 158.75 90)
-      (effects (font (size 1.27 1.27)) (justify left))
-    )
-    (property "Value" "TestPoint" (at 140.97 161.29 90)
-      (effects (font (size 1.27 1.27)) (justify left))
-    )
-    (property "Footprint" "footprints:TP_5014" (at 135.89 165.1 0)
-      (effects (font (size 1.27 1.27)) hide)
-    )
-    (property "Datasheet" "~" (at 135.89 165.1 0)
-      (effects (font (size 1.27 1.27)) hide)
-    )
-    (pin "1")
+  (symbol (lib_id "5014:5014") (at 140.97 160.02 0) (unit 1)
+    (in_bom yes) (on_board yes) (dnp no) (fields_autoplaced)
+    (property "Reference" "TP9" (at 143.51 158.75 0)
+      (effects (font (size 1.27 1.27)) (justify left))
+    )
+    (property "Value" "5014" (at 143.51 161.29 0)
+      (effects (font (size 1.27 1.27)) (justify left))
+    )
+    (property "Footprint" "footprints:TP_5014" (at 140.97 160.02 0)
+      (effects (font (size 1.27 1.27)) (justify bottom) hide)
+    )
+    (property "Datasheet" "" (at 140.97 160.02 0)
+      (effects (font (size 1.27 1.27)) hide)
+    )
+    (property "MF" "Keystone" (at 140.97 160.02 0)
+      (effects (font (size 1.27 1.27)) (justify bottom) hide)
+    )
+    (property "MAXIMUM_PACKAGE_HEIGHT" "8.13 mm" (at 140.97 160.02 0)
+      (effects (font (size 1.27 1.27)) (justify bottom) hide)
+    )
+    (property "Package" "None" (at 140.97 160.02 0)
+      (effects (font (size 1.27 1.27)) (justify bottom) hide)
+    )
+    (property "Price" "None" (at 140.97 160.02 0)
+      (effects (font (size 1.27 1.27)) (justify bottom) hide)
+    )
+    (property "Check_prices" "https://www.snapeda.com/parts/5014/Keystone/view-part/?ref=eda" (at 140.97 160.02 0)
+      (effects (font (size 1.27 1.27)) (justify bottom) hide)
+    )
+    (property "STANDARD" "Manufacturer Recommendations" (at 140.97 160.02 0)
+      (effects (font (size 1.27 1.27)) (justify bottom) hide)
+    )
+    (property "PARTREV" "F" (at 140.97 160.02 0)
+      (effects (font (size 1.27 1.27)) (justify bottom) hide)
+    )
+    (property "SnapEDA_Link" "https://www.snapeda.com/parts/5014/Keystone/view-part/?ref=snap" (at 140.97 160.02 0)
+      (effects (font (size 1.27 1.27)) (justify bottom) hide)
+    )
+    (property "MP" "5014" (at 140.97 160.02 0)
+      (effects (font (size 1.27 1.27)) (justify bottom) hide)
+    )
+    (property "Purchase-URL" "https://www.snapeda.com/api/url_track_click_mouser/?unipart_id=500798&manufacturer=Keystone&part_name=5014&search_term=	 pc test point multipurpos" (at 140.97 160.02 0)
+      (effects (font (size 1.27 1.27)) (justify bottom) hide)
+    )
+    (property "Description" "\nTest Point MultiPurpose THM H .445 Nylon 46 Insulated Yel PhosBronze/Silver | Keystone Electronics 5014\n" (at 140.97 160.02 0)
+      (effects (font (size 1.27 1.27)) (justify bottom) hide)
+    )
+    (property "MANUFACTURER" "Keystone Electronics" (at 140.97 160.02 0)
+      (effects (font (size 1.27 1.27)) (justify bottom) hide)
+    )
+    (property "Availability" "In Stock" (at 140.97 160.02 0)
+      (effects (font (size 1.27 1.27)) (justify bottom) hide)
+    )
+    (property "SNAPEDA_PN" "5010" (at 140.97 160.02 0)
+      (effects (font (size 1.27 1.27)) (justify bottom) hide)
+    )
+    (pin "TP")
     (instances
       (project "FufuS24"
@@
       (effects (font (size 1.27 1.27)))
     )
-    (property "Footprint" "footprints:TP_5014" (at 60.96 132.08 0)
-      (effects (font (size 1.27 1.27)) hide)
-    )
+    (property "Footprint" "footprints:FOD3150_footprint" (at 60.96 132.08 0)
+      (effects (font (size 1.27 1.27)) hide)
+    )
